File: Hardware/Diseño PCB/PWM/pwm.kicad_pcb (KiCad board)
At the start: 2 copper layers, 100.6 x 254.1 mm, 141 parts, among them J1 VE, J2 V_triag, J3 sense, J4 Vo, J5 pwm, Q1 IRF540N, Q2 IRF540N, U1 TL082, U2 IR2111

Commit message: PCB V2
Parts:
- removed the ? at (53.4, 105.1)
- removed the ? at (70.9, 177.9)
- removed the ? at (53.4, 194.1)
- removed the ? at (70.9, 266.9)
- removed the ? at (144.1, 260.1)
- removed the ? at (144.1, 171.1)
- removed the BC1 at (65.3, 261.8)
- removed the BC1 at (65.3, 172.8)
- removed the C1 at (69.6, 208.3)
- removed the C1 at (69.6, 119.3)
- removed the C2 at (125.7, 139.4)
- removed the C2 at (125.7, 228.4)
- removed the C3 at (123.8, 208.3)
- removed the C3 at (123.8, 119.3)
- removed the C4 at (115.6, 228.3)
- removed the C4 at (115.6, 139.3)
- removed the C5 at (101.6, 260.4)
- removed the C5 at (101.6, 171.4)
- removed the C6 at (92.1, 242.4)
- removed the C6 at (92.1, 153.4)
- removed the D1 at (141.0, 108.9)
- removed the D1 at (141.0, 197.9)
- removed D2 (x2): MBR735, Package_TO_SOT_THT:TO-220-2_Vertical
- removed the GND1 at (54.5, 233.2)
- removed the GND1 at (54.5, 144.2)
- removed the J1 at (57.7, 207.3)
- removed the J1 at (57.7, 118.3)
- removed the J2 at (107.9, 261.1)
- removed the J2 at (107.9, 172.1)
- removed the J3 at (140.9, 158.6)
- removed the J3 at (140.9, 247.6)
- removed the J4 at (142.1, 123.5)
- removed the J4 at (142.1, 212.5)
- removed the J5 at (111.1, 232.1)
- removed the J5 at (111.1, 143.1)
- removed the L1 at (85.5, 208.3)
- removed the L1 at (85.5, 119.3)
- removed the LM1 at (119.2, 252.9)
- removed the LM1 at (119.2, 163.9)
- removed the Q1 at (87.0, 107.6)
- removed the Q1 at (87.0, 196.6)
- removed the Q2 at (104.5, 107.6)
- removed the Q2 at (104.5, 196.6)
- removed the R1 at (110.5, 148.1)
- removed the R1 at (110.5, 237.1)
- removed the R10 at (61.8, 152.1)
- removed the R10 at (61.8, 241.1)
- removed the R11 at (107.0, 143.2)
- removed the R11 at (107.0, 232.2)
- removed the R12 at (70.6, 244.6)
- removed the R12 at (70.6, 155.6)
- removed the R13 at (70.8, 166.3)
- removed the R13 at (70.8, 255.3)
- removed the R14 at (128.9, 176.2)
- removed the R14 at (128.9, 265.2)
- removed the R15 at (107.7, 176.2)
- removed the R15 at (107.7, 265.2)
- removed the R16 at (118.4, 265.2)
- removed the R16 at (118.4, 176.2)
- removed the R17 at (139.4, 176.2)
- removed the R17 at (139.4, 265.2)
- removed the R2 at (99.1, 148.2)
- removed the R2 at (99.1, 237.2)
- removed the R3 at (132.6, 148.1)
- removed the R3 at (132.6, 237.1)
- removed the R4 at (140.9, 144.6)
- removed the R4 at (140.9, 233.6)
- removed the R5 at (145.9, 156.0)
- removed the R5 at (145.9, 245.0)
- removed the R6 at (145.9, 233.5)
- removed the R6 at (145.9, 144.5)
- removed the R7 at (138.2, 113.6)
- removed the R7 at (138.2, 202.6)
- removed the R8 at (61.8, 164.6)
- removed the R8 at (61.8, 253.6)
- removed the R9 at (61.8, 247.1)
- removed the R9 at (61.8, 158.1)
- removed the REF** at (146.9, 193.4)
- removed the REF** at (146.9, 104.4)
- removed the TL1 at (56.8, 261.5)
- removed the TL1 at (56.8, 172.5)
- removed the U1 at (102.2, 244.3)
- removed the U1 at (102.2, 155.3)
- removed the U2 at (79.6, 249.6)
- removed the U2 at (79.6, 160.6)
- removed the VEE1 at (54.5, 228.1)
- removed the VEE1 at (54.5, 139.1)
- removed the Vctrl_H1 at (81.0, 226.1)
- removed the Vctrl_H1 at (81.0, 137.1)
- removed the Vctrl_L1 at (89.3, 226.1)
- removed the Vctrl_L1 at (89.3, 137.1)
- removed the Vo1 at (142.7, 139.4)
- removed the Vo1 at (142.7, 228.4)
- added ?: , , F.Cu at (54.4, 106.0)
- added ?: , , F.Cu at (54.7, 194.7)
- added ?: , , F.Cu at (71.9, 178.8)
- added ?: , , F.Cu at (145.4, 260.7)
- added ?: , , F.Cu at (145.2, 172.0)
- added ?: , , F.Cu at (72.2, 267.4)
- added BC1: ~, Package_TO_SOT_THT:TO-92_HandSolder, F.Cu at (66.4, 173.7)
- added BC1: ~, Package_TO_SOT_THT:TO-92_HandSolder, F.Cu at (66.7, 262.4)
- added C1: 100u, Capacitor_THT:CP_Radial_D10.0mm_P2.50mm, F.Cu at (71.2, 208.8)
- added C1: 100u, Capacitor_THT:CP_Radial_D10.0mm_P2.50mm, F.Cu at (70.9, 120.2)
- added C2: 1n, Capacitor_THT:C_Disc_D6.0mm_W4.4mm_P5.00mm, F.Cu at (126.8, 139.5)
- added C2: 1n, Capacitor_THT:C_Disc_D6.0mm_W4.4mm_P5.00mm, F.Cu at (127.1, 228.2)
- added C3: 1n, Capacitor_THT:C_Disc_D3.0mm_W2.0mm_P2.50mm, F.Cu at (105.4, 200.2)
- added C3: 1n, Capacitor_THT:C_Disc_D3.0mm_W2.0mm_P2.50mm, F.Cu at (104.8, 25.5)
- added C3: 1n, Capacitor_THT:C_Disc_D3.0mm_W2.0mm_P2.50mm, F.Cu at (105.2, 111.5)
- added C4: 10n, Capacitor_THT:C_Disc_D6.0mm_W4.4mm_P5.00mm, F.Cu at (139.7, 262.2)
- added C4: 10n, Capacitor_THT:C_Disc_D6.0mm_W4.4mm_P5.00mm, F.Cu at (139.0, 87.5)
- added C4: 10n, Capacitor_THT:C_Disc_D6.0mm_W4.4mm_P5.00mm, F.Cu at (139.4, 173.5)
- added C5: 10n, Capacitor_THT:C_Disc_D6.0mm_W4.4mm_P5.00mm, F.Cu at (121.4, 145.0)
- added C5: 10n, Capacitor_THT:C_Disc_D6.0mm_W4.4mm_P5.00mm, F.Cu at (121.0, 59.0)
- added C5: 10n, Capacitor_THT:C_Disc_D6.0mm_W4.4mm_P5.00mm, F.Cu at (121.7, 233.7)
- added C6: 10n, Capacitor_THT:C_Disc_D6.0mm_W4.4mm_P5.00mm, F.Cu at (117.0, 228.2)
- added C6: 10n, Capacitor_THT:C_Disc_D6.0mm_W4.4mm_P5.00mm, F.Cu at (116.7, 139.5)
- added C7: 100u, Capacitor_THT:CP_Radial_D10.0mm_P2.50mm, F.Cu at (129.2, 210.7)
- added C7: 100u, Capacitor_THT:CP_Radial_D10.0mm_P2.50mm, F.Cu at (128.9, 122.0)
- added C8: 1n, Capacitor_THT:C_Disc_D6.0mm_W4.4mm_P5.00mm, F.Cu at (102.9, 260.9)
- added C8: 1n, Capacitor_THT:C_Disc_D6.0mm_W4.4mm_P5.00mm, F.Cu at (102.7, 172.3)
- added C9: 470n, Capacitor_THT:C_Disc_D6.0mm_W4.4mm_P5.00mm, F.Cu at (80.7, 226.2)
- added C9: 470n, Capacitor_THT:C_Disc_D6.0mm_W4.4mm_P5.00mm, F.Cu at (80.4, 137.5)
- added D1: D_Schottky, Diode_THT:D_DO-201AD_P12.70mm_Horizontal, F.Cu at (104.7, 39.0)
- added D1: D_Schottky, Diode_THT:D_DO-201AD_P12.70mm_Horizontal, F.Cu at (105.1, 125.0)
- added D1: D_Schottky, Diode_THT:D_DO-201AD_P12.70mm_Horizontal, F.Cu at (105.3, 213.7)
- added D3: MBR735, Diode_THT:D_A-405_P7.62mm_Horizontal, F.Cu at (92.5, 79.3)
- added D3: MBR735, Diode_THT:D_A-405_P7.62mm_Horizontal, F.Cu at (92.9, 165.3)
- added D3: MBR735, Diode_THT:D_A-405_P7.62mm_Horizontal, F.Cu at (93.2, 254.0)
- added D4: LED, LED_THT:LED_D4.0mm, F.Cu at (142.1, 109.8)
- added D4: LED, LED_THT:LED_D4.0mm, F.Cu at (142.3, 198.4)
- added D5: MBR735, Diode_THT:D_A-405_P7.62mm_Horizontal, F.Cu at (79.4, 148.5)
- added D5: MBR735, Diode_THT:D_A-405_P7.62mm_Horizontal, F.Cu at (79.7, 237.2)
- added GND1: GND, Connector_PinHeader_2.00mm:PinHeader_1x01_P2.00mm_Vertical, F.Cu at (55.9, 233.8)
- added GND1: GND, Connector_PinHeader_2.00mm:PinHeader_1x01_P2.00mm_Vertical, F.Cu at (55.6, 145.1)
- added J1: VE, TerminalBlock_Phoenix:TerminalBlock_Phoenix_MKDS-1,5-2_1x02_P5.00mm_Horizontal, F.Cu at (59.0, 207.9)
- added J1: VE, TerminalBlock_Phoenix:TerminalBlock_Phoenix_MKDS-1,5-2_1x02_P5.00mm_Horizontal, F.Cu at (58.8, 119.2)
- added J10: pwm, Connector_PinHeader_2.00mm:PinHeader_1x02_P2.00mm_Vertical, F.Cu at (112.2, 144.0)
- added J10: pwm, Connector_PinHeader_2.00mm:PinHeader_1x02_P2.00mm_Vertical, F.Cu at (112.4, 232.7)
- added J2: V_triag, Connector_PinHeader_2.00mm:PinHeader_1x01_P2.00mm_Vertical, F.Cu at (108.9, 173.0)
- added J2: V_triag, Connector_PinHeader_2.00mm:PinHeader_1x01_P2.00mm_Vertical, F.Cu at (109.2, 261.7)
- added J3: compensacion, Connector_PinHeader_2.00mm:PinHeader_1x02_P2.00mm_Vertical, F.Cu at (101.4, 136.5)
- added J3: compensacion, Connector_PinHeader_2.00mm:PinHeader_1x02_P2.00mm_Vertical, F.Cu at (101.7, 225.2)
- added J3: compensacion, Connector_PinHeader_2.00mm:PinHeader_1x02_P2.00mm_Vertical, F.Cu at (101.0, 50.5)
- added J4: sense, Connector_PinHeader_2.00mm:PinHeader_1x02_P2.00mm_Vertical, F.Cu at (133.5, 92.5)
- added J4: sense, Connector_PinHeader_2.00mm:PinHeader_1x02_P2.00mm_Vertical, F.Cu at (133.9, 178.5)
- added J4: sense, Connector_PinHeader_2.00mm:PinHeader_1x02_P2.00mm_Vertical, F.Cu at (134.2, 267.2)
- added J5: Snubber, Connector_PinHeader_2.00mm:PinHeader_1x02_P2.00mm_Vertical, F.Cu at (107.4, 106.0)
- added J5: Snubber, Connector_PinHeader_2.00mm:PinHeader_1x02_P2.00mm_Vertical, F.Cu at (107.0, 20.0)
- added J5: Snubber, Connector_PinHeader_2.00mm:PinHeader_1x02_P2.00mm_Vertical, F.Cu at (107.7, 194.7)
- added J6: sense, Connector_PinHeader_2.00mm:PinHeader_1x02_P2.00mm_Vertical, F.Cu at (142.9, 139.5)
- added J6: sense, Connector_PinHeader_2.00mm:PinHeader_1x02_P2.00mm_Vertical, F.Cu at (143.2, 228.2)
- added J7: compensacion, Connector_PinHeader_2.00mm:PinHeader_1x02_P2.00mm_Vertical, F.Cu at (101.7, 228.2)
- added J7: compensacion, Connector_PinHeader_2.00mm:PinHeader_1x02_P2.00mm_Vertical, F.Cu at (101.4, 139.5)
- added J7: compensacion, Connector_PinHeader_2.00mm:PinHeader_1x02_P2.00mm_Vertical, F.Cu at (101.0, 53.5)
- added J8: V_triag, Connector_PinHeader_2.00mm:PinHeader_1x02_P2.00mm_Vertical, F.Cu at (110.2, 152.8)
- added J8: V_triag, Connector_PinHeader_2.00mm:PinHeader_1x02_P2.00mm_Vertical, F.Cu at (109.8, 66.8)
- added J8: V_triag, Connector_PinHeader_2.00mm:PinHeader_1x02_P2.00mm_Vertical, F.Cu at (110.4, 241.4)
- added J9: Vo, TerminalBlock_Phoenix:TerminalBlock_Phoenix_MKDS-1,5-2_1x02_P5.00mm_Horizontal, F.Cu at (143.4, 213.0)
- added J9: Vo, TerminalBlock_Phoenix:TerminalBlock_Phoenix_MKDS-1,5-2_1x02_P5.00mm_Horizontal, F.Cu at (143.1, 124.4)
- added L1: 50u, Bobinados:EE19, F.Cu at (81.5, 118.0)
- added L1: 50u, Bobinados:EE19, F.Cu at (81.7, 206.6)
- added LM1: LM319, Package_DIP:DIP-14_W7.62mm_Socket, F.Cu at (120.5, 253.4)
- added LM1: LM319, Package_DIP:DIP-14_W7.62mm_Socket, F.Cu at (120.2, 164.8)
- added Q1: IRF540N, Package_TO_SOT_THT:TO-220-3_Vertical, F.Cu at (85.4, 124.0)
- added Q1: IRF540N, Package_TO_SOT_THT:TO-220-3_Vertical, F.Cu at (85.7, 212.7)
- added Q2: IRF540N, Package_TO_SOT_THT:TO-220-3_Vertical, F.Cu at (96.8, 212.7)
- added Q2: IRF540N, Package_TO_SOT_THT:TO-220-3_Vertical, F.Cu at (96.5, 124.0)
- added Q9: BC557, Package_TO_SOT_THT:TO-92_Wide, F.Cu at (88.1, 266.4)
- added Q9: BC557, Package_TO_SOT_THT:TO-92_Wide, F.Cu at (87.5, 91.8)
- added Q9: BC557, Package_TO_SOT_THT:TO-92_Wide, F.Cu at (87.9, 177.8)
- added R1: 10k, Resistor_THT:R_Axial_DIN0204_L3.6mm_D1.6mm_P7.62mm_Horizontal, F.Cu at (111.6, 149.0)
- added R1: 10k, Resistor_THT:R_Axial_DIN0204_L3.6mm_D1.6mm_P7.62mm_Horizontal, F.Cu at (111.8, 237.7)
- added R10: 1k, Resistor_THT:R_Axial_DIN0204_L3.6mm_D1.6mm_P7.62mm_Horizontal, F.Cu at (143.5, 70.2)
- added R10: 1k, Resistor_THT:R_Axial_DIN0204_L3.6mm_D1.6mm_P7.62mm_Horizontal, F.Cu at (144.2, 244.9)
- added R10: 1k, Resistor_THT:R_Axial_DIN0204_L3.6mm_D1.6mm_P7.62mm_Horizontal, F.Cu at (143.9, 156.2)
- added R11: 1k, Resistor_THT:R_Axial_DIN0204_L3.6mm_D1.6mm_P7.62mm_Horizontal, F.Cu at (63.1, 254.2)
- added R11: 1k, Resistor_THT:R_Axial_DIN0204_L3.6mm_D1.6mm_P7.62mm_Horizontal, F.Cu at (62.8, 165.5)
- added R12: 10k, Resistor_THT:R_Axial_DIN0204_L3.6mm_D1.6mm_P7.62mm_Horizontal, F.Cu at (146.0, 77.8)
- added R12: 10k, Resistor_THT:R_Axial_DIN0204_L3.6mm_D1.6mm_P7.62mm_Horizontal, F.Cu at (146.4, 163.8)
- added R12: 10k, Resistor_THT:R_Axial_DIN0204_L3.6mm_D1.6mm_P7.62mm_Horizontal, F.Cu at (146.7, 252.5)
- added R13: 10k, Resistor_THT:R_Axial_DIN0204_L3.6mm_D1.6mm_P7.62mm_Horizontal, F.Cu at (63.1, 247.7)
- added R13: 10k, Resistor_THT:R_Axial_DIN0204_L3.6mm_D1.6mm_P7.62mm_Horizontal, F.Cu at (62.8, 159.0)
- added R14: 10k, Resistor_THT:R_Axial_DIN0204_L3.6mm_D1.6mm_P7.62mm_Horizontal, F.Cu at (63.1, 241.7)
- added R14: 10k, Resistor_THT:R_Axial_DIN0204_L3.6mm_D1.6mm_P7.62mm_Horizontal, F.Cu at (62.8, 153.0)
- added R15: 1k, Resistor_THT:R_Axial_DIN0204_L3.6mm_D1.6mm_P7.62mm_Horizontal, F.Cu at (108.3, 232.8)
- added R15: 1k, Resistor_THT:R_Axial_DIN0204_L3.6mm_D1.6mm_P7.62mm_Horizontal, F.Cu at (108.0, 144.1)
- added R16: 100k, Resistor_THT:R_Axial_DIN0204_L3.6mm_D1.6mm_P7.62mm_Horizontal, F.Cu at (71.7, 156.5)
- added R16: 100k, Resistor_THT:R_Axial_DIN0204_L3.6mm_D1.6mm_P7.62mm_Horizontal, F.Cu at (72.0, 245.2)
- added R17: 100k, Resistor_THT:R_Axial_DIN0204_L3.6mm_D1.6mm_P7.62mm_Horizontal, F.Cu at (72.1, 255.9)
- added R17: 100k, Resistor_THT:R_Axial_DIN0204_L3.6mm_D1.6mm_P7.62mm_Horizontal, F.Cu at (71.8, 167.2)
- added R18: 1k, Resistor_THT:R_Axial_DIN0204_L3.6mm_D1.6mm_P7.62mm_Horizontal, F.Cu at (80.4, 246.7)
- added R18: 1k, Resistor_THT:R_Axial_DIN0204_L3.6mm_D1.6mm_P7.62mm_Horizontal, F.Cu at (79.7, 72.0)
- added R18: 1k, Resistor_THT:R_Axial_DIN0204_L3.6mm_D1.6mm_P7.62mm_Horizontal, F.Cu at (80.1, 158.0)
- added R19: 1k, Resistor_THT:R_Axial_DIN0204_L3.6mm_D1.6mm_P7.62mm_Horizontal, F.Cu at (80.1, 161.2)
- added R19: 1k, Resistor_THT:R_Axial_DIN0204_L3.6mm_D1.6mm_P7.62mm_Horizontal, F.Cu at (80.4, 249.8)
- added R19: 1k, Resistor_THT:R_Axial_DIN0204_L3.6mm_D1.6mm_P7.62mm_Horizontal, F.Cu at (79.7, 75.2)
- added R2: 30k, Resistor_THT:R_Axial_DIN0204_L3.6mm_D1.6mm_P7.62mm_Horizontal, F.Cu at (100.1, 149.1)
- added R2: 30k, Resistor_THT:R_Axial_DIN0204_L3.6mm_D1.6mm_P7.62mm_Horizontal, F.Cu at (100.4, 237.8)
- added R20: 10k, Resistor_THT:R_Axial_DIN0204_L3.6mm_D1.6mm_P7.62mm_Horizontal, F.Cu at (80.4, 255.9)
- added R20: 10k, Resistor_THT:R_Axial_DIN0204_L3.6mm_D1.6mm_P7.62mm_Horizontal, F.Cu at (80.1, 167.2)
- added R20: 10k, Resistor_THT:R_Axial_DIN0204_L3.6mm_D1.6mm_P7.62mm_Horizontal, F.Cu at (79.7, 81.2)
- added R21: 5k6, Resistor_THT:R_Axial_DIN0204_L3.6mm_D1.6mm_P7.62mm_Horizontal, F.Cu at (119.9, 260.7)
- added R21: 5k6, Resistor_THT:R_Axial_DIN0204_L3.6mm_D1.6mm_P7.62mm_Horizontal, F.Cu at (119.6, 172.0)
- added R22: 1k, Resistor_THT:R_Axial_DIN0204_L3.6mm_D1.6mm_P7.62mm_Horizontal, F.Cu at (79.7, 78.2)
- added R22: 1k, Resistor_THT:R_Axial_DIN0204_L3.6mm_D1.6mm_P7.62mm_Horizontal, F.Cu at (80.4, 252.9)
- added R22: 1k, Resistor_THT:R_Axial_DIN0204_L3.6mm_D1.6mm_P7.62mm_Horizontal, F.Cu at (80.1, 164.2)
- added R23: 33k, Resistor_THT:R_Axial_DIN0204_L3.6mm_D1.6mm_P7.62mm_Horizontal, F.Cu at (108.8, 177.1)
- added R23: 33k, Resistor_THT:R_Axial_DIN0204_L3.6mm_D1.6mm_P7.62mm_Horizontal, F.Cu at (109.0, 265.7)
- added R24: 100k, Resistor_THT:R_Axial_DIN0204_L3.6mm_D1.6mm_P7.62mm_Horizontal, F.Cu at (119.6, 174.5)
- added R24: 100k, Resistor_THT:R_Axial_DIN0204_L3.6mm_D1.6mm_P7.62mm_Horizontal, F.Cu at (119.9, 263.2)
- added R25: 10k, Resistor_THT:R_Axial_DIN0204_L3.6mm_D1.6mm_P7.62mm_Horizontal, F.Cu at (80.4, 259.3)
- added R25: 10k, Resistor_THT:R_Axial_DIN0204_L3.6mm_D1.6mm_P7.62mm_Horizontal, F.Cu at (80.1, 170.6)
- added R25: 10k, Resistor_THT:R_Axial_DIN0204_L3.6mm_D1.6mm_P7.62mm_Horizontal, F.Cu at (79.7, 84.6)
- added R26: 1k, Resistor_THT:R_Axial_DIN0204_L3.6mm_D1.6mm_P7.62mm_Horizontal, F.Cu at (119.9, 265.7)
- added R26: 1k, Resistor_THT:R_Axial_DIN0204_L3.6mm_D1.6mm_P7.62mm_Horizontal, F.Cu at (119.6, 177.0)
- added R3: 33k, Resistor_THT:R_Axial_DIN0204_L3.6mm_D1.6mm_P7.62mm_Horizontal, F.Cu at (133.9, 237.7)
- added R3: 33k, Resistor_THT:R_Axial_DIN0204_L3.6mm_D1.6mm_P7.62mm_Horizontal, F.Cu at (133.7, 149.0)
- added R4: 56k, Resistor_THT:R_Axial_DIN0204_L3.6mm_D1.6mm_P7.62mm_Horizontal, F.Cu at (144.7, 231.9)
- added R4: 56k, Resistor_THT:R_Axial_DIN0204_L3.6mm_D1.6mm_P7.62mm_Horizontal, F.Cu at (144.4, 143.2)
- added R5: 10k, Resistor_THT:R_Axial_DIN0204_L3.6mm_D1.6mm_P7.62mm_Horizontal, F.Cu at (141.9, 143.2)
- added R5: 10k, Resistor_THT:R_Axial_DIN0204_L3.6mm_D1.6mm_P7.62mm_Horizontal, F.Cu at (142.2, 231.9)
- added R6: 33k, Resistor_THT:R_Axial_DIN0204_L3.6mm_D1.6mm_P7.62mm_Horizontal, F.Cu at (146.7, 178.5)
- added R6: 33k, Resistor_THT:R_Axial_DIN0204_L3.6mm_D1.6mm_P7.62mm_Horizontal, F.Cu at (147.0, 267.2)
- added R6: 33k, Resistor_THT:R_Axial_DIN0204_L3.6mm_D1.6mm_P7.62mm_Horizontal, F.Cu at (146.3, 92.5)
- added R7: 56k, Resistor_THT:R_Axial_DIN0204_L3.6mm_D1.6mm_P7.62mm_Horizontal, F.Cu at (147.2, 231.9)
- added R7: 56k, Resistor_THT:R_Axial_DIN0204_L3.6mm_D1.6mm_P7.62mm_Horizontal, F.Cu at (146.9, 143.2)
- added R8: ~, Resistor_THT:R_Axial_DIN0414_L11.9mm_D4.5mm_P15.24mm_Horizontal, F.Cu at (105.1, 207.2)
- added R8: ~, Resistor_THT:R_Axial_DIN0414_L11.9mm_D4.5mm_P15.24mm_Horizontal, F.Cu at (104.8, 118.5)
- added R8: ~, Resistor_THT:R_Axial_DIN0414_L11.9mm_D4.5mm_P15.24mm_Horizontal, F.Cu at (104.4, 32.5)
- added R9: ~, Resistor_THT:R_Axial_DIN0204_L3.6mm_D1.6mm_P7.62mm_Horizontal, F.Cu at (139.3, 114.5)
- added R9: ~, Resistor_THT:R_Axial_DIN0204_L3.6mm_D1.6mm_P7.62mm_Horizontal, F.Cu at (139.6, 203.2)
- added REF**: EE25, Bobinados:EE25, F.Cu at (82.4, 119.5)
- added REF**: MountingHole_3.2mm_M3, MountingHole:MountingHole_3.2mm_M3, F.Cu at (147.9, 105.2)
- added REF**: EE25, Bobinados:EE25, F.Cu at (82.0, 33.5)
- added REF**: EE25, Bobinados:EE25, F.Cu at (82.7, 208.2)
- added REF**: MountingHole_3.2mm_M3, MountingHole:MountingHole_3.2mm_M3, F.Cu at (148.2, 193.9)
- added RV1: Preset, Potentiometer_THT:Potentiometer_Bourns_3386P_Vertical, F.Cu at (120.2, 198.7)
- added RV1: Preset, Potentiometer_THT:Potentiometer_Bourns_3386P_Vertical, F.Cu at (119.5, 24.0)
- added RV1: Preset, Potentiometer_THT:Potentiometer_Bourns_3386P_Vertical, F.Cu at (119.9, 110.0)
- added TL1: TL431LP, Package_TO_SOT_THT:TO-92_HandSolder, F.Cu at (57.9, 173.4)
- added TL1: TL431LP, Package_TO_SOT_THT:TO-92_HandSolder, F.Cu at (58.2, 262.1)
- added TL2: TL431LP, Package_TO_SOT_THT:TO-92_HandSolder, F.Cu at (82.0, 91.5)
- added TL2: TL431LP, Package_TO_SOT_THT:TO-92_HandSolder, F.Cu at (82.4, 177.5)
- added TL2: TL431LP, Package_TO_SOT_THT:TO-92_HandSolder, F.Cu at (82.6, 266.2)
- added U1: TL082, Package_DIP:DIP-8_W7.62mm_Socket, F.Cu at (103.6, 244.9)
- added U1: TL082, Package_DIP:DIP-8_W7.62mm_Socket, F.Cu at (103.3, 156.2)
- added U2: IR2111, Package_DIP:DIP-8_W7.62mm_Socket, F.Cu at (85.4, 232.5)
- added U2: IR2111, Package_DIP:DIP-8_W7.62mm_Socket, F.Cu at (85.1, 143.8)
- added VEE1: VEE, Connector_PinHeader_2.00mm:PinHeader_1x01_P2.00mm_Vertical, F.Cu at (55.9, 228.7)
- added VEE1: VEE, Connector_PinHeader_2.00mm:PinHeader_1x01_P2.00mm_Vertical, F.Cu at (55.6, 140.0)
- added Vctrl_H1: Vctrl_H, Connector_PinHeader_2.00mm:PinHeader_1x01_P2.00mm_Vertical, F.Cu at (68.9, 135.5)
- added Vctrl_H1: Vctrl_H, Connector_PinHeader_2.00mm:PinHeader_1x01_P2.00mm_Vertical, F.Cu at (69.2, 224.2)
- added Vctrl_L1: Vctrl_L, Connector_PinHeader_2.00mm:PinHeader_1x01_P2.00mm_Vertical, F.Cu at (92.7, 147.0)
- added Vctrl_L1: Vctrl_L, Connector_PinHeader_2.00mm:PinHeader_1x01_P2.00mm_Vertical, F.Cu at (92.9, 235.7)
- added Vo1: Vo, Connector_PinHeader_2.00mm:PinHeader_1x01_P2.00mm_Vertical, F.Cu at (146.7, 228.2)
- added Vo1: Vo, Connector_PinHeader_2.00mm:PinHeader_1x01_P2.00mm_Vertical, F.Cu at (146.4, 139.5)
- C9: renamed from C6; value 10u -> 470n
- D5: renamed from D2; footprint Package_TO_SOT_THT:TO-220-2_Vertical -> Diode_THT:D_A-405_P7.62mm_Horizontal
- L1: footprint Inductor_THT:L_Axial_L20.0mm_D8.0mm_P25.40mm_Horizontal -> Bobinados:EE19
- moved D5 29.0 mm to (79.0, 62.5), turned to 0 degrees
- moved C9 21.1 mm to (80.0, 51.5), turned to -90 degrees
- moved R26 20.8 mm to (119.2, 91.0)
- moved J6 20.0 mm to (142.5, 53.5), turned to -90 degrees
- moved U2 18.2 mm to (84.7, 57.8), turned to 90 degrees
- moved Q2 17.9 mm to (96.1, 38.0), turned to 180 degrees
- moved Q1 15.7 mm to (85.0, 38.0), turned to 180 degrees
- moved R5 14.6 mm to (141.5, 57.2)
- moved Vctrl_H1 13.4 mm to (68.5, 49.5)
- moved R21 11.5 mm to (119.2, 86.0)
- moved Vctrl_L1 9.32 mm to (92.2, 61.0)
- moved L1 5.61 mm to (81.0, 32.0)
- moved C7 4.45 mm to (128.5, 36.0)
- moved R4 3.40 mm to (144.0, 57.2)
- moved Vo1 2.77 mm to (146.0, 53.5)
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- renumbered C4 to C6, C3 to C7, C5 to C8, D1 to D4, J5 to J10, J3 to J6, J4 to J9, R8 to R11, R9 to R13, R10 to R14, R11 to R15, R12 to R16, R13 to R17, R14 to R21, R15 to R23, R16 to R24, R17 to R26, R6 to R7, R7 to R9
Connections:
- C6 pad 2: Net-(LM1B-+) -> Net-(J7-Pin_2)
- LM1 pad 10: /V_triag -> Net-(J8-Pin_1)
- R15 pad 2: /VEE -> /Vcc5
- U1 pad 1: Net-(LM1B-+) -> Net-(D3-A)
- U1 pad 3: /Vmed -> Net-(J4-Pin_1)
Routing:
- net Net-(J10-Pin_1): track 428.4 -> 88.8 mm, vias 0 -> 6
- net Net-(D3-A): track 0.00 -> 308.8 mm, vias 0 -> 12
- net Net-(LM1B-+): track 294.9 -> 48.8 mm
- net /Vctrl_L: track 232.4 -> 73.8 mm
- net /VEE: track 624.7 -> 478.7 mm, vias 6 -> 0
- net /Vctrl_H: track 240.6 -> 105.7 mm
- net Net-(J4-Pin_1): track 0.00 -> 126.3 mm, vias 0 -> 6
- net GND: track 603.9 -> 485.0 mm
- net Net-(J3-Pin_2): track 202.3 -> 313.6 mm
- net /Vcc3: track 0.00 -> 101.9 mm
- net /Vs: track 255.3 -> 351.7 mm
- net Net-(J7-Pin_2): track 0.00 -> 86.4 mm
- net /Vcc5: track 388.5 -> 472.8 mm, vias 18 -> 24
- net /V_triag: track 179.1 -> 102.4 mm
- net /PWM: track 148.8 -> 217.2 mm
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Other:
- board size 100.6 x 254.1 mm -> 100.7 x 254.7 mm
- board text added: "Comp"
- board text added: "Fuente Buck"
- board text added: "Grupo 7:"
- board text added: "PWM LIM"
- board text added: "Snubber"
- board text added: "VMED"
- board text added: "Vmed"
- board text added: "Vmuestra"
- board text added: "Vtriag"
- board text removed: "Grupo 7: Regulador Buck"
- board text removed: "Señales de Control"
