File: Hardware/Diseño PCB/PWM/pwm.kicad_pcb (KiCad board)
At the start: 2 copper layers, 100.7 x 254.7 mm, 210 parts, among them J1 VE, J10 pwm, J2 V_triag, J3 compensacion, J4 sense, J5 Snubber, J6 sense, J7 compensacion, J8 V_triag, J9 Vo, Q1 IRF540N, Q2 IRF540N, Q9 BC557, U1 TL082, U2 IR2111

Commit message: PCB V2
Parts:
- removed the ? at (54.4, 106.0)
- removed the ? at (54.7, 194.7)
- removed the ? at (71.9, 178.8)
- removed the ? at (145.4, 260.7)
- removed the ? at (145.2, 172.0)
- removed the ? at (72.2, 267.4)
- removed the BC1 at (66.4, 173.7)
- removed the BC1 at (66.7, 262.4)
- removed the C1 at (71.2, 208.8)
- removed the C1 at (70.9, 120.2)
- removed the C2 at (126.8, 139.5)
- removed the C2 at (127.1, 228.2)
- removed the C3 at (105.4, 200.2)
- removed the C3 at (105.2, 111.5)
- removed the C4 at (139.7, 262.2)
- removed the C4 at (139.4, 173.5)
- removed the C5 at (121.4, 145.0)
- removed the C5 at (121.7, 233.7)
- removed the C6 at (117.0, 228.2)
- removed the C6 at (116.7, 139.5)
- removed the C7 at (129.2, 210.7)
- removed the C7 at (128.9, 122.0)
- removed the C8 at (102.9, 260.9)
- removed the C8 at (102.7, 172.3)
- removed the C9 at (80.7, 226.2)
- removed the C9 at (80.4, 137.5)
- removed the D1 at (105.1, 125.0)
- removed the D1 at (105.3, 213.7)
- removed the D3 at (92.9, 165.3)
- removed the D3 at (93.2, 254.0)
- removed the D4 at (142.1, 109.8)
- removed the D4 at (142.3, 198.4)
- removed the D5 at (79.4, 148.5)
- removed the D5 at (79.7, 237.2)
- removed the GND1 at (55.9, 233.8)
- removed the GND1 at (55.6, 145.1)
- removed the J1 at (59.0, 207.9)
- removed the J1 at (58.8, 119.2)
- removed the J10 at (112.2, 144.0)
- removed the J10 at (112.4, 232.7)
- removed the J2 at (108.9, 173.0)
- removed the J2 at (109.2, 261.7)
- removed the J3 at (101.4, 136.5)
- removed the J3 at (101.7, 225.2)
- removed the J4 at (133.9, 178.5)
- removed the J4 at (134.2, 267.2)
- removed the J5 at (107.4, 106.0)
- removed the J5 at (107.7, 194.7)
- removed the J6 at (142.9, 139.5)
- removed the J6 at (143.2, 228.2)
- removed the J7 at (101.7, 228.2)
- removed the J7 at (101.4, 139.5)
- removed the J8 at (110.2, 152.8)
- removed the J8 at (110.4, 241.4)
- removed the J9 at (143.4, 213.0)
- removed the J9 at (143.1, 124.4)
- removed the L1 at (81.5, 118.0)
- removed the L1 at (81.7, 206.6)
- removed the LM1 at (120.5, 253.4)
- removed the LM1 at (120.2, 164.8)
- removed the Q1 at (85.4, 124.0)
- removed the Q1 at (85.7, 212.7)
- removed the Q2 at (96.8, 212.7)
- removed the Q2 at (96.5, 124.0)
- removed the Q9 at (88.1, 266.4)
- removed the Q9 at (87.9, 177.8)
- removed the R1 at (111.6, 149.0)
- removed the R1 at (111.8, 237.7)
- removed the R10 at (144.2, 244.9)
- removed the R10 at (143.9, 156.2)
- removed the R11 at (63.1, 254.2)
- removed the R11 at (62.8, 165.5)
- removed the R12 at (146.4, 163.8)
- removed the R12 at (146.7, 252.5)
- removed the R13 at (63.1, 247.7)
- removed the R13 at (62.8, 159.0)
- removed the R14 at (63.1, 241.7)
- removed the R14 at (62.8, 153.0)
- removed the R15 at (108.3, 232.8)
- removed the R15 at (108.0, 144.1)
- removed the R16 at (71.7, 156.5)
- removed the R16 at (72.0, 245.2)
- removed the R17 at (72.1, 255.9)
- removed the R17 at (71.8, 167.2)
- removed the R18 at (80.4, 246.7)
- removed the R18 at (80.1, 158.0)
- removed the R19 at (80.1, 161.2)
- removed the R19 at (80.4, 249.8)
- removed the R2 at (100.1, 149.1)
- removed the R2 at (100.4, 237.8)
- removed the R20 at (80.4, 255.9)
- removed the R20 at (80.1, 167.2)
- removed the R21 at (119.9, 260.7)
- removed the R21 at (119.6, 172.0)
- removed the R22 at (80.4, 252.9)
- removed the R22 at (80.1, 164.2)
- removed the R23 at (108.8, 177.1)
- removed the R23 at (109.0, 265.7)
- removed the R24 at (119.6, 174.5)
- removed the R24 at (119.9, 263.2)
- removed the R25 at (80.4, 259.3)
- removed the R25 at (80.1, 170.6)
- removed the R26 at (119.9, 265.7)
- removed the R26 at (119.6, 177.0)
- removed the R3 at (133.9, 237.7)
- removed the R3 at (133.7, 149.0)
- removed the R4 at (144.7, 231.9)
- removed the R4 at (144.4, 143.2)
- removed the R5 at (141.9, 143.2)
- removed the R5 at (142.2, 231.9)
- removed the R6 at (146.7, 178.5)
- removed the R6 at (147.0, 267.2)
- removed the R7 at (147.2, 231.9)
- removed the R7 at (146.9, 143.2)
- removed the R8 at (105.1, 207.2)
- removed the R8 at (104.8, 118.5)
- removed the R9 at (139.3, 114.5)
- removed the R9 at (139.6, 203.2)
- removed the REF** at (82.4, 119.5)
- removed the REF** at (147.9, 105.2)
- removed the REF** at (82.7, 208.2)
- removed the REF** at (148.2, 193.9)
- removed the RV1 at (120.2, 198.7)
- removed the RV1 at (119.9, 110.0)
- removed the TL1 at (57.9, 173.4)
- removed the TL1 at (58.2, 262.1)
- removed the TL2 at (82.4, 177.5)
- removed the TL2 at (82.6, 266.2)
- removed the U1 at (103.6, 244.9)
- removed the U1 at (103.3, 156.2)
- removed the U2 at (85.4, 232.5)
- removed the U2 at (85.1, 143.8)
- removed the VEE1 at (55.9, 228.7)
- removed the VEE1 at (55.6, 140.0)
- removed the Vctrl_H1 at (68.9, 135.5)
- removed the Vctrl_H1 at (69.2, 224.2)
- removed the Vctrl_L1 at (92.7, 147.0)
- removed the Vctrl_L1 at (92.9, 235.7)
- removed the Vo1 at (146.7, 228.2)
- removed the Vo1 at (146.4, 139.5)
- added D2: 5V, Diode_THT:D_DO-34_SOD68_P7.62mm_Horizontal, F.Cu at (138.0, 65.9)
Routing:
- net GND: track 485.0 -> 161.7 mm, vias 12 -> 4
- net /VEE: track 478.7 -> 159.6 mm
- net /Vcc5: track 472.8 -> 157.6 mm, vias 24 -> 8
- net /Vs: track 351.7 -> 117.2 mm, vias 6 -> 2
- net /Vo: track 328.5 -> 109.5 mm, vias 6 -> 2
- net Net-(J3-Pin_2): track 313.6 -> 104.5 mm
- net Net-(D3-A): track 308.8 -> 102.9 mm, vias 12 -> 4
- net /Vmed: track 283.8 -> 94.6 mm, vias 18 -> 6
- net /v_muestra: track 222.3 -> 74.1 mm, vias 6 -> 2
- net /PWM: track 217.2 -> 72.4 mm, vias 6 -> 2
- net Net-(U1B--): track 161.3 -> 53.8 mm, vias 6 -> 2
- net /V_cuad: track 140.8 -> 46.9 mm
- net Net-(J4-Pin_1): track 126.3 -> 42.1 mm, vias 6 -> 2
- net /Vctrl_H: track 105.7 -> 35.2 mm, vias 6 -> 2
- net /V_triag: track 102.4 -> 34.1 mm
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Other:
- board size 100.7 x 254.7 mm -> 100 x 80 mm
