File: Hardware/Diseño PCB/PWM/pwm.kicad_pcb (KiCad board)
At the start: 2 copper layers, 100 x 80 mm, 71 parts, among them J1 VE, J10 pwm, J2 V_triag, J3 compensacion, J4 sense, J5 Snubber, J6 sense, J7 compensacion, J8 V_triag, J9 Vo, Q1 IRF540N, Q2 IRF540N, Q9 BC557, U1 TL082, U2 IR2111

Commit message: Avances en informe general
Parts:
- moved Q9 87.9 mm to (91.8, 179.6)
- moved U1 87.9 mm to (107.2, 158.1)
- moved ? 87.9 mm to (149.1, 173.8)
- moved ? 87.9 mm to (75.8, 180.6)
- moved ? 87.9 mm to (58.3, 107.8)
- moved BC1 87.9 mm to (70.3, 175.5)
- moved C1 87.9 mm to (74.8, 122.0)
- moved C2 87.9 mm to (130.7, 141.3)
- moved C3 87.9 mm to (109.1, 113.3)
- moved C4 87.9 mm to (143.3, 175.3)
- moved C5 87.9 mm to (125.3, 146.8)
- moved C6 87.9 mm to (120.6, 141.3)
- moved C7 87.9 mm to (132.8, 123.8)
- moved C8 87.9 mm to (106.6, 174.1)
- moved C9 87.9 mm to (84.3, 139.3)
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