File: Hardware/Diseño PCB/PWM/pwm.kicad_sch (KiCad schematic)
At the start: 63 parts, among them J1 VE, J2 V_triag, J3 sense, J4 Vo, J5 pwm, J6 Snubber, J7 sense, J8 V_triag, Q1 IRF540N, Q2 IRF540N, U1 TL082, U2 IR2111

Commit message: PCB V2
Parts:
- removed BC2: (no value), Package_TO_SOT_THT:TO-92_HandSolder, symbol Transistor_BJT:BC546
- removed R23, R24: 100k, Resistor_THT:R_Axial_DIN0204_L3.6mm_D1.6mm_P7.62mm_Horizontal, symbol Device:R
- added C5: 10n, Capacitor_THT:C_Disc_D6.0mm_W4.4mm_P5.00mm, symbol Device:C
- added J3, J7: compensacion, Connector_PinHeader_2.00mm:PinHeader_1x02_P2.00mm_Vertical, symbol Connector:Conn_01x02_Pin
- added Q9: BC557, Package_TO_SOT_THT:TO-92_Wide, symbol Transistor_BJT:BC557
- added R22: 1k, Resistor_THT:R_Axial_DIN0204_L3.6mm_D1.6mm_P7.62mm_Horizontal, symbol Device:R
- added R25: 10k, Resistor_THT:R_Axial_DIN0204_L3.6mm_D1.6mm_P7.62mm_Horizontal, symbol Device:R
- C3: renamed from C8; footprint Capacitor_THT:CP_Radial_D10.0mm_P2.50mm -> Capacitor_THT:C_Disc_D3.0mm_W2.0mm_P2.50mm
- D1: renamed from D3; footprint (none) -> Diode_THT:D_DO-201AD_P12.70mm_Horizontal
- D2: renamed from D5; footprint (none) -> Diode_THT:D_DO-34_SOD68_P7.62mm_Horizontal
- D3: renamed from D4; footprint Package_TO_SOT_THT:TO-220-2_Vertical -> Diode_THT:D_A-405_P7.62mm_Horizontal
- D5: renamed from D2; footprint Package_TO_SOT_THT:TO-220-2_Vertical -> Diode_THT:D_A-405_P7.62mm_Horizontal
- L1: footprint Inductor_THT:L_Axial_L20.0mm_D8.0mm_P25.40mm_Horizontal -> Bobinados:EE19
- R19: renamed from R21; value 10k -> 1k
- R8: renamed from R18; footprint Resistor_THT:R_Axial_DIN0204_L3.6mm_D1.6mm_P7.62mm_Horizontal -> Resistor_THT:R_Axial_DIN0414_L11.9mm_D4.5mm_P15.24mm_Horizontal
- gave numbers to parts that had none: 1
- renumbered C7 to C4, C4 to C6, C3 to C7, C5 to C8, C6 to C9, D1 to D4, J5 to J10, J7 to J4, J6 to J5, J3 to J6, J4 to J9, R8 to R11, R25 to R12, R9 to R13, R10 to R14, R11 to R15, R12 to R16, R13 to R17, R20 to R18, R22 to R20, R14 to R21, R15 to R23, R16 to R24, R17 to R26, R19 to R6, R6 to R7, R7 to R9, RV2 to RV1
Connections:
- net GND: now also R25.2
- net Vcc3: now also R18.2, Q9.3 (E), R22.1
- net v_muestra: now also J3.1 (Pin_1)
- net at D3.2 (A), R10.1, U1.1: now also J7.1 (Pin_1); no longer C6.2
- net at C2.2, R2.2, R3.1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: now also C5.1, J3.2 (Pin_2)
- net at TL2.3 (K): now also Q9.2 (B), R22.2; no longer R18.2
- new net: C5.2, C6.2, J7.2 (Pin_2)
- new net: Q9.1 (C), R25.1
Other:
- note added: "Limitador PWM"
- moved on the sheet: R18, R19, R20, TL2

Commit message: Avances en informe general
Changed lines of the file:
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@@
 		(in_pos_files yes)
 		(dnp no)
-		(fields_autoplaced yes)
 		(property "Reference" "C1"
-			(at 59.69 31.7499 0)
+			(at 47.498 32.766 0)
 			(show_name no)
 			(do_not_autoplace no)
@@
 		)
 		(property "Value" "100u"
-			(at 59.69 34.2899 0)
+			(at 47.752 34.798 0)
 			(show_name no)
 			(do_not_autoplace no)
@@
 		(in_pos_files yes)
 		(dnp no)
-		(fields_autoplaced yes)
 		(property "Reference" "Q1"
-			(at 69.85 15.24 90)
-			(show_name no)
-			(do_not_autoplace no)
+			(at 73.914 24.13 90)
+			(show_name no)
+			(do_not_autoplace no)
